Commit message: Add noise + change model

File: hector_sensors_description/urdf/generic_camera_plus.urdf.xacro (robot description, xacro)
@@ -17,5 +17,5 @@
         <origin xyz="0 0 0" rpy="0 0 0" />
         <geometry>
-        <mesh filename="package://hector_sensors_description/meshes/hokuyo_utm30lx/hokuyo_utm_30lx$(optenv TEST_SELF_FILTER).dae"/>
+        <mesh filename="package://hector_sensors_description/meshes/hokuyo_utm30lx/hokuyo_utm30lx.dae"/>
       </geometry>
       </visual>
@@ -38,7 +38,12 @@
           </image>
           <clip>
-            <near>0.1</near>
-            <far>100</far>
+            <near>0.02</near>
+            <far>300</far>
           </clip>
+          <noise>
+            <type>gaussian</type>
+            <mean>0.0</mean>
+            <stddev>0.007</stddev>
+        </noise>
         </camera>
         <plugin name="${name}_camera_controller" filename="libgazebo_ros_camera.so">
